File: Bus_switch.kicad_sch (KiCad schematic)
At the start: 15 parts, among them J3 Conn_01x04_Pin, U1 SN74CB3Q3384APW

Commit message: Schematic
Parts:
- renumbered C1 to C3, D3 to D1, R2 to R1, R4 to R10, R1 to R11, R3 to R2, R5 to R3, R6 to R4, R7 to R5, R8 to R6, R9 to R7, R10 to R8, R11 to R9, U1 to U2
