File: Bus_switch.kicad_sch (KiCad schematic)
At the start: 15 parts, among them J3 Conn_01x04_Pin, U2 SN74CB3Q3384APW

Commit message: Schematic touchup
Parts:
- removed R1, R2, R3, R5, R6, R7, R9: 10kΩ, PCM_JLCPCB:R_0402, symbol PCM_JLCPCB-Resistors:0402,10kΩ
