File: CH32V003.kicad_sch (KiCad schematic)
At the start: 11 parts, among them J6 WCH Link, J7 Program, U8 CH32V003FxPx, X2 X322525MOB4SI

Commit message: Schematic
Parts:
- renumbered C6 to C16, C5 to C17, C4 to C18, D7 to D9, J6 to J8, J7 to J9, R17 to R51, R31 to R52, U8 to U7, X2 to X1
Changed lines of the file:
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@@
 		(dnp no)
 		(fields_autoplaced yes)
-		(property "Reference" "#PWR060"
+		(property "Reference" "#PWR0102"
 			(at 40.64 166.37 0)
 			(hide yes)
@@
 			(project "MMS3_hat_templates"
 				(path "/6596548a-44e0-46d8-8624-fd71cf4a3e17/f4f5cc42-4af7-4189-bf2e-976157de876a"
-					(reference "#PWR060")
+					(reference "#PWR0102")
 					(unit 1)
 				)
@@
 		(dnp no)
 		(fields_autoplaced yes)
-		(property "Reference" "#PWR068"
+		(property "Reference" "#PWR0110"
 			(at 162.56 102.87 0)
 			(hide yes)
@@
 			(project "MMS3_hat_templates"
 				(path "/6596548a-44e0-46d8-8624-fd71cf4a3e17/f4f5cc42-4af7-4189-bf2e-976157de876a"
-					(reference "#PWR068")
+					(reference "#PWR0110")
 					(unit 1)
 				)
@@
 		(in_pos_files yes)
 		(dnp no)
-		(property "Reference" "#PWR078"
+		(property "Reference" "#PWR0111"
 			(at 209.55 158.75 0)
 			(hide yes)
@@
 			(project "MMS3_hat_templates"
 				(path "/6596548a-44e0-46d8-8624-fd71cf4a3e17/f4f5cc42-4af7-4189-bf2e-976157de876a"
-					(reference "#PWR078")
+					(reference "#PWR0111")
 					(unit 1)
 				)
@@
 		(in_pos_files yes)
 		(dnp no)
-		(property "Reference" "#PWR061"
+		(property "Reference" "#PWR0103"
 			(at 46.99 132.08 0)
 			(hide yes)
@@
 			(project "MMS3_hat_templates"
 				(path "/6596548a-44e0-46d8-8624-fd71cf4a3e17/f4f5cc42-4af7-4189-bf2e-976157de876a"
-					(reference "#PWR061")
+					(reference "#PWR0103")
 					(unit 1)
 				)
@@
 		(dnp no)
 		(fields_autoplaced yes)
-		(property "Reference" "C4"
+		(property "Reference" "C18"
 			(at 198.12 148.5899 0)
 			(show_name no)
@@
 			(project "MMS3_hat_templates"
 				(path "/6596548a-44e0-46d8-8624-fd71cf4a3e17/f4f5cc42-4af7-4189-bf2e-976157de876a"
-					(reference "C4")
+					(reference "C18")
 					(unit 1)
 				)
@@
 		(dnp no)
 		(fields_autoplaced yes)
-		(property "Reference" "#PWR065"
+		(property "Reference" "#PWR0107"
 			(at 127 138.43 0)
 			(hide yes)
@@
 			(project "MMS3_hat_templates"
 				(path "/6596548a-44e0-46d8-8624-fd71cf4a3e17/f4f5cc42-4af7-4189-bf2e-976157de876a"
-					(reference "#PWR065")
+					(reference "#PWR0107")
 					(unit 1)
 				)
@@
 		(dnp no)
 		(fields_autoplaced yes)
-		(property "Reference" "U8"
+		(property "Reference" "U7"
 			(at 164.7033 53.34 0)
 			(show_name no)
@@
 			(project "MMS3_hat_templates"
 				(path "/6596548a-44e0-46d8-8624-fd71cf4a3e17/f4f5cc42-4af7-4189-bf2e-976157de876a"
-					(reference "U8")
+					(reference "U7")
 					(unit 1)
 				)
@@
 		(dnp no)
 		(fields_autoplaced yes)
-		(property "Reference" "#PWR058"
+		(property "Reference" "#PWR0100"
 			(at 49.53 168.91 0)
 			(hide yes)
@@
 			(project "MMS3_hat_templates"
 				(path "/6596548a-44e0-46d8-8624-fd71cf4a3e17/f4f5cc42-4af7-4189-bf2e-976157de876a"
-					(reference "#PWR058")
+					(reference "#PWR0100")
 					(unit 1)
 				)
@@
 		(dnp no)
 		(fields_autoplaced yes)
-		(property "Reference" "C6"
+		(property "Reference" "C16"
 			(at 129.54 35.5599 0)
 			(show_name no)
@@
 			(project "MMS3_hat_templates"
 				(path "/6596548a-44e0-46d8-8624-fd71cf4a3e17/f4f5cc42-4af7-4189-bf2e-976157de876a"
-					(reference "C6")
+					(reference "C16")
 					(unit 1)
 				)
@@
 		(dnp no)
 		(fields_autoplaced yes)
-		(property "Reference" "#PWR063"
+		(property "Reference" "#PWR0105"
 			(at 127 34.29 0)
 			(hide yes)
@@
 			(project "MMS3_hat_templates"
 				(path "/6596548a-44e0-46d8-8624-fd71cf4a3e17/f4f5cc42-4af7-4189-bf2e-976157de876a"
-					(reference "#PWR063")
+					(reference "#PWR0105")
 					(unit 1)
 				)
@@
 		(in_pos_files yes)
 		(dnp no)
-		(property "Reference" "#PWR066"
+		(property "Reference" "#PWR0108"
 			(at 154.94 154.94 0)
 			(hide yes)
@@
 			(project "MMS3_hat_templates"
 				(path "/6596548a-44e0-46d8-8624-fd71cf4a3e17/f4f5cc42-4af7-4189-bf2e-976157de876a"
-					(reference "#PWR066")
+					(reference "#PWR0108")
 					(unit 1)
 				)
@@
 		(dnp no)
 		(fields_autoplaced yes)
-		(property "Reference" "#PWR0101"
+		(property "Reference" "#PWR0112"
 			(at 248.92 92.71 0)
 			(hide yes)
@@
 			(project "MMS3_hat_templates"
 				(path "/6596548a-44e0-46d8-8624-fd71cf4a3e17/f4f5cc42-4af7-4189-bf2e-976157de876a"
-					(reference "#PWR0101")
+					(reference "#PWR0112")
 					(unit 1)
 				)
@@
 		(dnp yes)
 		(fields_autoplaced yes)
-		(property "Reference" "J6"
+		(property "Reference" "J8"
 			(at 57.15 154.94 0)
 			(show_name no)
@@
 			(project "MMS3_hat_templates"
 				(path "/6596548a-44e0-46d8-8624-fd71cf4a3e17/f4f5cc42-4af7-4189-bf2e-976157de876a"
-					(reference "J6")
+					(reference "J8")
 					(unit 1)
 				)
@@
 		(dnp no)
 		(fields_autoplaced yes)
-		(property "Reference" "R31"
+		(property "Reference" "R52"
 			(at 251.46 59.6899 0)
 			(show_name no)
@@
 			(project "MMS3_hat_templates"
 				(path "/6596548a-44e0-46d8-8624-fd71cf4a3e17/f4f5cc42-4af7-4189-bf2e-976157de876a"
-					(reference "R31")
+					(reference "R52")
 					(unit 1)
 				)
@@
 		(dnp no)
 		(fields_autoplaced yes)
-		(property "Reference" "C5"
+		(property "Reference" "C17"
 			(at 187.96 148.5899 0)
 			(show_name no)
@@
 			(project "MMS3_hat_templates"
 				(path "/6596548a-44e0-46d8-8624-fd71cf4a3e17/f4f5cc42-4af7-4189-bf2e-976157de876a"
-					(reference "C5")
+					(reference "C17")
 					(unit 1)
 				)
@@
 		(dnp no)
 		(fields_autoplaced yes)
-		(property "Reference" "J7"
+		(property "Reference" "J9"
 			(at 72.39 133.3499 0)
 			(show_name no)
@@
 			(project "MMS3_hat_templates"
 				(path "/6596548a-44e0-46d8-8624-fd71cf4a3e17/f4f5cc42-4af7-4189-bf2e-976157de876a"
-					(reference "J7")
+					(reference "J9")
 					(unit 1)
 				)
@@
 		(dnp no)
 		(fields_autoplaced yes)
-		(property "Reference" "D7"
+		(property "Reference" "D9"
 			(at 251.46 72.2946 0)
 			(show_name no)
@@
 			(project "MMS3_hat_templates"
 				(path "/6596548a-44e0-46d8-8624-fd71cf4a3e17/f4f5cc42-4af7-4189-bf2e-976157de876a"
-					(reference "D7")
+					(reference "D9")
 					(unit 1)
 				)
@@
 		(dnp no)
 		(fields_autoplaced yes)
-		(property "Reference" "#PWR064"
+		(property "Reference" "#PWR0106"
 			(at 127 53.34 0)
 			(hide yes)
@@
 			(project "MMS3_hat_templates"
 				(path "/6596548a-44e0-46d8-8624-fd71cf4a3e17/f4f5cc42-4af7-4189-bf2e-976157de876a"
-					(reference "#PWR064")
+					(reference "#PWR0106")
 					(unit 1)
 				)
@@
 		(dnp no)
 		(fields_autoplaced yes)
-		(property "Reference" "R17"
+		(property "Reference" "R51"
 			(at 129.54 140.9699 0)
 			(show_name no)
@@
 			(project "MMS3_hat_templates"
 				(path "/6596548a-44e0-46d8-8624-fd71cf4a3e17/f4f5cc42-4af7-4189-bf2e-976157de876a"
-					(reference "R17")
+					(reference "R51")
 					(unit 1)
 				)
@@
 		(dnp no)
 		(fields_autoplaced yes)
-		(property "Reference" "X2"
+		(property "Reference" "X1"
 			(at 172.72 129.54 0)
 			(show_name no)
@@
 			(project "MMS3_hat_templates"
 				(path "/6596548a-44e0-46d8-8624-fd71cf4a3e17/f4f5cc42-4af7-4189-bf2e-976157de876a"
-					(reference "X2")
+					(reference "X1")
 					(unit 1)
 				)
@@
 		(in_pos_files yes)
 		(dnp no)
-		(property "Reference" "#PWR062"
+		(property "Reference" "#PWR0104"
 			(at 57.15 137.16 0)
 			(hide yes)
@@
 			(project "MMS3_hat_templates"
 				(path "/6596548a-44e0-46d8-8624-fd71cf4a3e17/f4f5cc42-4af7-4189-bf2e-976157de876a"
-					(reference "#PWR062")
+					(reference "#PWR0104")
 					(unit 1)
 				)
@@
 		(dnp no)
 		(fields_autoplaced yes)
-		(property "Reference" "#PWR067"
+		(property "Reference" "#PWR0109"
 			(at 162.56 53.34 0)
 			(hide yes)
@@
 			(project "MMS3_hat_templates"
 				(path "/6596548a-44e0-46d8-8624-fd71cf4a3e17/f4f5cc42-4af7-4189-bf2e-976157de876a"
-					(reference "#PWR067")
+					(reference "#PWR0109")
 					(unit 1)
 				)
@@
 		(dnp no)
 		(fields_autoplaced yes)
-		(property "Reference" "#PWR059"
+		(property "Reference" "#PWR0101"
 			(at 49.53 171.45 0)
 			(hide yes)
@@
 			(project "MMS3_hat_templates"
 				(path "/6596548a-44e0-46d8-8624-fd71cf4a3e17/f4f5cc42-4af7-4189-bf2e-976157de876a"
-					(reference "#PWR059")
+					(reference "#PWR0101")
 					(unit 1)
 				)
