File: MMS3_hat_templates.kicad_pcb (KiCad board)
At the start: 2 copper layers, 100 x 50 mm, 35 parts, among them J1 Chainbus in, J2 Chainbus Out, J3 Conn_01x04_Pin, J4 AMASS XT60 Male, J5 AMASS XT60 Female, U1 SN74CB3Q3384APW, U2 M24C64, U4 AMS1117

Commit message: Schematic
Parts:
- added C17: 10uF, PCM_JLCPCB:C_0603, F.Cu at (235.2, 26.8)
- added C19: 10uF, PCM_JLCPCB:C_0603, F.Cu at (235.2, 29.0)
- added C20: 100nF, PCM_JLCPCB:C_0603, F.Cu at (61.9, 43.9)
- added C21: 100nF, PCM_JLCPCB:C_0603, F.Cu at (64.9, 43.9)
- added C22: 3.3nF, PCM_JLCPCB:C_0603, F.Cu at (49.6, 35.5)
- added C23: 100nF, PCM_JLCPCB:C_0603, F.Cu at (45.6, 21.6)
- added C24: 100nF, PCM_JLCPCB:C_0603, F.Cu at (44.8, 19.4)
- added C31: 100nF, PCM_JLCPCB:C_0603, F.Cu at (247.6, 63.0)
- added C4: 12pF, PCM_JLCPCB:C_0603, F.Cu at (269.5, 16.6)
- added C5: 12pF, PCM_JLCPCB:C_0603, F.Cu at (269.5, 18.9)
- added C50: 100uF, Capacitor_SMD:CP_Elec_10x10, F.Cu at (71.3, 35.6)
- added C51: 100uF, Capacitor_SMD:CP_Elec_10x10, F.Cu at (54.0, 48.1)
- added C6: 100nF, PCM_JLCPCB:C_0603, F.Cu at (269.5, 21.1)
- added C7: 100nF, PCM_JLCPCB:C_0603, F.Cu at (276.2, 46.9)
- added D10: SS510C, SS510C:SMC_L7.1-W6.2-LS8.1-RD, F.Cu at (238.7, 21.9)
- added D4: SS510C, SS510C:SMC_L7.1-W6.2-LS8.1-RD, F.Cu at (32.7, 40.6)
- added D5: SS510C, SS510C:SMC_L7.1-W6.2-LS8.1-RD, F.Cu at (77.1, 62.1)
- added D6: SS510C, SS510C:SMC_L7.1-W6.2-LS8.1-RD, F.Cu at (70.6, 50.6)
- added D7: Red, PCM_JLCPCB:D_0603, F.Cu at (279.3, 19.7)
- added D8: Red, PCM_JLCPCB:D_0603, F.Cu at (79.1, 52.8)
- added D9: Red, PCM_JLCPCB:D_0603, F.Cu at (243.6, 63.2)
- added H1: M2.5 Mount, MountingHole:MountingHole_2.7mm_M2.5_DIN965_Pad_TopOnly, F.Cu at (32.1, 61.5)
- added H3: M2.5 mount, MountingHole:MountingHole_2.7mm_M2.5, F.Cu at (32.1, 19.5)
- added H5: M2.5 mount, MountingHole:MountingHole_2.7mm_M2.5, F.Cu at (53.1, 21.5)
- added H7: ~, PCM_JLCPCB:Hole_Tooling_JLCPCB, F.Cu at (29.2, 64.5)
- added H9: ~, PCM_JLCPCB:Hole_Tooling_JLCPCB, F.Cu at (29.1, 16.5)
- added J10: LED connector, Connector_JST:JST_XH_S4B-XH-A_1x04_P2.50mm_Horizontal, F.Cu at (249.9, 35.5)
- added J11: LED connector, Connector_JST:JST_XH_S4B-XH-A_1x04_P2.50mm_Horizontal, F.Cu at (254.6, 9.19)
- added J12: LED connector, Connector_JST:JST_XH_S4B-XH-A_1x04_P2.50mm_Horizontal, F.Cu at (228.6, 35.5)
- added J4: AMASS XT60 Male, XT60:AMASS_XT60PW-M_1x02_P7.20mm_Horizontal, F.Cu at (48.5, 57.8)
- added J5: AMASS XT60 Female, XT60:AMASS_XT60PW-F_1x02_P7.20mm_Horizontal, F.Cu at (58.0, 57.8)
- added J7: Program, Connector_PinHeader_2.54mm:PinHeader_1x03_P2.54mm_Vertical, F.Cu at (269.8, 8.14)
- added J8: Conn_01x03_Pin, Connector_PinHeader_2.54mm:PinHeader_1x03_P2.54mm_Vertical, F.Cu at (63.3, 47.3)
- added J9: LED connector, Connector_JST:JST_XH_S4B-XH-A_1x04_P2.50mm_Horizontal, F.Cu at (271.3, 35.5)
- added L1: 100uH 4A, Inductor_SMD:L_Sunlord_SWRB1207S, F.Cu at (41.7, 30.1)
- added Q10: 2N7002K, PCM_JLCPCB:Q_SOT-23, F.Cu at (248.6, 8.25)
- added Q11: 2N7002K, PCM_JLCPCB:Q_SOT-23, F.Cu at (248.6, 12.9)
- added Q12: 2N7002K, PCM_JLCPCB:Q_SOT-23, F.Cu at (248.6, 17.5)
- added Q13: 2N7002K, PCM_JLCPCB:Q_SOT-23, F.Cu at (222.7, 34.6)
- added Q14: 2N7002K, PCM_JLCPCB:Q_SOT-23, F.Cu at (222.7, 39.2)
- added Q15: 2N7002K, PCM_JLCPCB:Q_SOT-23, F.Cu at (222.7, 43.8)
- added Q3: 2N7002K, PCM_JLCPCB:Q_SOT-23, F.Cu at (265.4, 34.6)
- added Q4: 2N7002K, PCM_JLCPCB:Q_SOT-23, F.Cu at (265.4, 39.2)
- added Q6: 2N7002K, PCM_JLCPCB:Q_SOT-23, F.Cu at (244.0, 34.6)
- added Q7: 2N7002K, PCM_JLCPCB:Q_SOT-23, F.Cu at (244.0, 39.2)
- added Q8: 2N7002K, PCM_JLCPCB:Q_SOT-23, F.Cu at (265.4, 43.8)
- added Q9: 2N7002K, PCM_JLCPCB:Q_SOT-23, F.Cu at (244.0, 43.8)
- added R10: 33kΩ, PCM_JLCPCB:R_0402, F.Cu at (61.4, 44.9)
- added R11: 33kΩ, PCM_JLCPCB:R_0402, F.Cu at (64.6, 44.9)
- added R15: 510Ω, PCM_JLCPCB:R_0402, F.Cu at (49.9, 32.3)
- added R16: 510Ω, PCM_JLCPCB:R_0402, F.Cu at (49.9, 33.3)
- added R17: 10kΩ, PCM_JLCPCB:R_0402, F.Cu at (47.0, 22.0)
- added R21: 33kΩ, PCM_JLCPCB:R_0402, F.Cu at (221.7, 6.78)
- added R22: 33kΩ, PCM_JLCPCB:R_0402, F.Cu at (221.7, 8.62)
- added R23: 1kΩ, PCM_JLCPCB:R_0402, F.Cu at (221.7, 10.5)
- added R24: 18.7k, PCM_JLCPCB:R_0402, F.Cu at (221.7, 12.3)
- added R25: 16.5k, PCM_JLCPCB:R_0402, F.Cu at (221.7, 14.2)
- added R26: 9.53k, PCM_JLCPCB:R_0402, F.Cu at (221.7, 16.0)
- added R27: 5.11k, PCM_JLCPCB:R_0402, F.Cu at (221.7, 17.9)
- added R28: 33kΩ, PCM_JLCPCB:R_0402, F.Cu at (221.7, 19.7)
- added R29: 33kΩ, PCM_JLCPCB:R_0402, F.Cu at (221.7, 21.6)
- added R30: 10kΩ, PCM_JLCPCB:R_0402, F.Cu at (272.9, 46.7)
- added R31: 330Ω, PCM_JLCPCB:R_0402, F.Cu at (280.6, 14.8)
- added R32: 200Ω, PCM_JLCPCB:R_0603, F.Cu at (269.6, 46.9)
- added R33: 10kΩ, PCM_JLCPCB:R_0402, F.Cu at (272.9, 48.5)
- added R34: 200Ω, PCM_JLCPCB:R_0603, F.Cu at (269.6, 49.1)
- added R35: 10kΩ, PCM_JLCPCB:R_0402, F.Cu at (243.0, 55.4)
- added R36: 10kΩ, PCM_JLCPCB:R_0402, F.Cu at (243.0, 57.3)
- added R37: 10kΩ, PCM_JLCPCB:R_0402, F.Cu at (243.0, 59.1)
- added R38: 10kΩ, PCM_JLCPCB:R_0402, F.Cu at (243.0, 61.0)
- added R39: 10kΩ, PCM_JLCPCB:R_0402, F.Cu at (245.8, 55.4)
- added R40: 10kΩ, PCM_JLCPCB:R_0402, F.Cu at (245.8, 57.3)
- added R41: 10kΩ, PCM_JLCPCB:R_0402, F.Cu at (245.8, 59.1)
- added R42: 10kΩ, PCM_JLCPCB:R_0402, F.Cu at (245.8, 61.0)
- added R43: 10kΩ, PCM_JLCPCB:R_0402, F.Cu at (248.7, 55.4)
- added R44: 10kΩ, PCM_JLCPCB:R_0402, F.Cu at (248.7, 57.3)
- added R45: 10kΩ, PCM_JLCPCB:R_0402, F.Cu at (248.7, 59.1)
- added R46: 10kΩ, PCM_JLCPCB:R_0402, F.Cu at (248.7, 61.0)
- added R47: 10kΩ, PCM_JLCPCB:R_0402, F.Cu at (272.9, 50.4)
- added R48: 10kΩ, PCM_JLCPCB:R_0402, F.Cu at (251.5, 46.7)
- added R49: 200Ω, PCM_JLCPCB:R_0603, F.Cu at (269.6, 51.4)
- added R51: 200Ω, PCM_JLCPCB:R_0603, F.Cu at (248.3, 46.9)
- added R52: 10kΩ, PCM_JLCPCB:R_0402, F.Cu at (251.5, 48.5)
- added R53: 200Ω, PCM_JLCPCB:R_0603, F.Cu at (248.3, 49.1)
- added R54: 10kΩ, PCM_JLCPCB:R_0402, F.Cu at (251.5, 50.4)
- added R55: 200Ω, PCM_JLCPCB:R_0603, F.Cu at (248.3, 51.4)
- added R56: 10kΩ, PCM_JLCPCB:R_0402, F.Cu at (256.2, 20.3)
- added R57: 200Ω, PCM_JLCPCB:R_0603, F.Cu at (252.9, 20.5)
- added R58: 10kΩ, PCM_JLCPCB:R_0402, F.Cu at (256.2, 22.2)
- added R59: 200Ω, PCM_JLCPCB:R_0603, F.Cu at (252.9, 22.8)
- added R60: 10kΩ, PCM_JLCPCB:R_0402, F.Cu at (256.2, 24.0)
- added R61: 200Ω, PCM_JLCPCB:R_0603, F.Cu at (252.9, 25.0)
- added R62: 10kΩ, PCM_JLCPCB:R_0402, F.Cu at (230.2, 46.7)
- added R63: 200Ω, PCM_JLCPCB:R_0603, F.Cu at (226.9, 46.9)
- added R64: 10kΩ, PCM_JLCPCB:R_0402, F.Cu at (230.2, 48.5)
- added R65: 200Ω, PCM_JLCPCB:R_0603, F.Cu at (226.9, 49.1)
- added R66: 10kΩ, PCM_JLCPCB:R_0402, F.Cu at (230.2, 50.4)
- added R67: 200Ω, PCM_JLCPCB:R_0603, F.Cu at (226.9, 51.4)
- added S1: Tactile Button, 160gf, PCM_JLCPCB:SW_TS-1088-AR02016, F.Cu at (275.6, 16.1)
- added SW1: SW_DIP_x04, Button_Switch_THT:SW_DIP_SPSTx04_Slide_6.7x11.72mm_W7.62mm_P2.54mm_LowProfile, F.Cu at (53.9, 39.5)
- added TP8: TestPoint, TestPoint:TestPoint_Pad_D1.0mm, F.Cu at (55.4, 29.2)
- added U5: PCA9685PW,118, easyeda2kicad:TSSOP-28_L9.7-W4.4-P0.65-LS6.4-TL, F.Cu at (41.9, 47.9)
- added U6: AMS1117, PCM_JLCPCB:SOT-223-3_L6.5-W3.4-P2.30-LS7.0-BR, F.Cu at (227.7, 22.2)
- added U7: LM2596HVS-ADJRG, Package_TO_SOT_SMD:TO-263-5_TabPin3, F.Cu at (233.8, 12.0)
- added U8: CH32V003FxPx, PCM_JLCPCB:TSSOP-20_4.4x6.5mm_P0.65mm, F.Cu at (276.9, 9.88)
- added X2: X322525MOB4SI, PCM_JLCPCB:OSC-SMD_4P-L3.2-W2.5-BL, F.Cu at (274.7, 20.4)
Connections:
- net /Bus_switch/Chainbus.SCL renamed /Chainbus.SCL
- net /Bus_switch/Chainbus.SDA renamed /Chainbus.SDA
- net /Power Connector/VIN_BRD renamed /Buck Regulator/VIN_BRD
Routing:
- net U_reg: track 0.00 -> 61.4 mm
- net (no net): track 0.00 -> 55.6 mm, vias 0 -> 35
- net GND: track 16.6 -> 57.7 mm, vias 24 -> 71
- net /Bus_switch/SEL1: track 82.8 -> 108.6 mm
- net Vin: track 0.00 -> 12.5 mm
- net Net-(D5-A): track 0.00 -> 11.6 mm
- net Net-(C23-Pad2): track 0.00 -> 10.1 mm
- net /Buck Regulator/sw-vin: track 0.00 -> 7.80 mm
- net Net-(R25-Pad1): track 0.00 -> 6.67 mm
- net Net-(D10-A): track 0.00 -> 6.46 mm
- net /Buck Regulator/sw: track 0.00 -> 6.06 mm
- net Net-(C20-Pad2): track 0.00 -> 5.53 mm
- net Net-(D6-A): track 0.00 -> 4.63 mm
- net +5V: track 58.4 -> 62.5 mm, vias 3 -> 7
- net /Interboard_connector/SEL2: track 2.59 -> 5.43 mm, vias 1 -> 2
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- added copper zone on B.Cu, net (none)
- added copper zone on F.Cu, net (none)
- added copper zone on F.Cu, net /Buck Regulator/sw
- added copper zone on F.Cu, net /Buck Regulator/sw-vin
- added copper zone on F.Cu, net Net-(C20-Pad2)
- added copper zone on F.Cu, net Net-(C23-Pad2)
- added copper zone on F.Cu, net U_reg
Other:
- copper layers 2 -> 4
- board text added: "J1"
- board text added: "J2"

Commit message: Schematic touchup
Parts:
- removed C21, C23, C24, C31, C7: 100nF, PCM_JLCPCB:C_0603
- removed C22: 3.3nF, PCM_JLCPCB:C_0603
- removed C50, C51: 100uF, Capacitor_SMD:CP_Elec_10x10
- removed D10, D5: SS510C, SS510C:SMC_L7.1-W6.2-LS8.1-RD
- removed D7, D8: Red, PCM_JLCPCB:D_0603
- removed the H1 at (32.1, 61.5)
- removed the H3 at (32.1, 19.5)
- removed the H5 at (53.1, 21.5)
- removed the H7 at (29.2, 64.5)
- removed the H9 at (29.1, 16.5)
- removed J12: LED connector, Connector_JST:JST_XH_S4B-XH-A_1x04_P2.50mm_Horizontal
- removed the J4 at (48.5, 57.8)
- removed the J5 at (58.0, 57.8)
- removed J8: Conn_01x03_Pin, Connector_PinHeader_2.54mm:PinHeader_1x03_P2.54mm_Vertical
- removed R1: 330Ω, PCM_JLCPCB:R_0402
- removed the R10 at (61.4, 44.9)
- removed the R10 at (152.0, 109.5)
- removed the R11 at (64.6, 44.9)
- removed the R11 at (149.1, 111.2)
- removed R2, R3, R37, R41, R5, R56, R6, R64, R7, R9: 10kΩ, PCM_JLCPCB:R_0402
- removed R29: 33kΩ, PCM_JLCPCB:R_0402
- removed SW1: SW_DIP_x04, Button_Switch_THT:SW_DIP_SPSTx04_Slide_6.7x11.72mm_W7.62mm_P2.54mm_LowProfile
- removed TP8: TestPoint, TestPoint:TestPoint_Pad_D1.0mm
- removed U5: PCA9685PW,118, easyeda2kicad:TSSOP-28_L9.7-W4.4-P0.65-LS6.4-TL
- removed U8: CH32V003FxPx, PCM_JLCPCB:TSSOP-20_4.4x6.5mm_P0.65mm
- removed X2: X322525MOB4SI, PCM_JLCPCB:OSC-SMD_4P-L3.2-W2.5-BL
- added C10: 100nF, PCM_JLCPCB:C_0603, F.Cu at (1.43, 24.3)
- added C11: 100nF, PCM_JLCPCB:C_0603, F.Cu at (1.43, 26.6)
- added C12: 3.3nF, PCM_JLCPCB:C_0603, F.Cu at (1.43, 28.8)
- added C13: 100nF, PCM_JLCPCB:C_0603, F.Cu at (1.43, 31.1)
- added C14: 100nF, PCM_JLCPCB:C_0603, F.Cu at (1.43, 33.3)
- added C15: 100uF, Capacitor_SMD:CP_Elec_10x10, F.Cu at (6.81, 17.3)
- added C3: 100nF, PCM_JLCPCB:C_0603, F.Cu at (64.5, 59.6)
- added C9: 100uF, Capacitor_SMD:CP_Elec_10x10, F.Cu at (6.81, 5.42)
- added D2: M7, PCM_JLCPCB:D_SMA, F.Cu at (62.6, 12.2)
- added J6: LED connector, Connector_JST:JST_XH_S4B-XH-A_1x04_P2.50mm_Horizontal, F.Cu at (125.7, 132.8)
- added Q1: AO3400A, PCM_JLCPCB:Q_SOT-23, F.Cu at (35.7, 1.90)
- added Q16: MMBT5401 200-300, PCM_JLCPCB:Q_SOT-23, F.Cu at (40.6, 31.3)
- added Q17: AO3400A, PCM_JLCPCB:Q_SOT-23, F.Cu at (40.6, 36.0)
- added Q18: AO3400A, PCM_JLCPCB:Q_SOT-23, F.Cu at (1.95, 43.5)
- added Q19: MMBT2222A 1P, PCM_JLCPCB:Q_SOT-23, F.Cu at (40.6, 40.6)
- added Q2: MMBT2222A 1P, PCM_JLCPCB:Q_SOT-23, F.Cu at (35.7, 6.53)
- added Q20: MMBT2222A 1P, PCM_JLCPCB:Q_SOT-23, F.Cu at (45.5, 31.3)
- added Q21: MMBT5401 200-300, PCM_JLCPCB:Q_SOT-23, F.Cu at (45.5, 36.0)
- added Q22: MMBT2222A 1P, PCM_JLCPCB:Q_SOT-23, F.Cu at (45.5, 40.6)
- added Q23: MMBT2222A 1P, PCM_JLCPCB:Q_SOT-23, F.Cu at (50.4, 31.3)
- added Q24: MMBT5401 200-300, PCM_JLCPCB:Q_SOT-23, F.Cu at (50.4, 36.0)
- added Q25: 2N7002K, PCM_JLCPCB:Q_SOT-23, F.Cu at (167.0, 114.3)
- added Q26: 2N7002K, PCM_JLCPCB:Q_SOT-23, F.Cu at (167.0, 110.8)
- added Q27: AO3400A, PCM_JLCPCB:Q_SOT-23, F.Cu at (50.4, 11.2)
- added Q28: MMBT2222A 1P, PCM_JLCPCB:Q_SOT-23, F.Cu at (1.95, 48.1)
- added Q29: MMBT2222A 1P, PCM_JLCPCB:Q_SOT-23, F.Cu at (6.83, 38.9)
- added Q30: MMBT5401 200-300, PCM_JLCPCB:Q_SOT-23, F.Cu at (6.83, 43.5)
- added Q31: AO3400A, PCM_JLCPCB:Q_SOT-23, F.Cu at (50.4, 40.6)
- added Q32: AO3400A, PCM_JLCPCB:Q_SOT-23, F.Cu at (6.83, 48.1)
- added Q33: MMBT2222A 1P, PCM_JLCPCB:Q_SOT-23, F.Cu at (11.7, 38.9)
- added Q34: MMBT2222A 1P, PCM_JLCPCB:Q_SOT-23, F.Cu at (11.7, 43.5)
- added Q35: MMBT5401 200-300, PCM_JLCPCB:Q_SOT-23, F.Cu at (11.7, 48.1)
- added Q36: MMBT2222A 1P, PCM_JLCPCB:Q_SOT-23, F.Cu at (16.6, 38.9)
- added Q37: MMBT2222A 1P, PCM_JLCPCB:Q_SOT-23, F.Cu at (16.6, 43.5)
- added Q38: MMBT5401 200-300, PCM_JLCPCB:Q_SOT-23, F.Cu at (16.6, 48.1)
- added Q5: AO3400A, PCM_JLCPCB:Q_SOT-23, F.Cu at (35.7, 31.3)
- added R10: 10kΩ, PCM_JLCPCB:R_0402, F.Cu at (97.8, 40.7)
- added R11: 330Ω, PCM_JLCPCB:R_0402, F.Cu at (67.8, 59.4)
- added R12: 510Ω, PCM_JLCPCB:R_0402, F.Cu at (173.6, 120.5)
- added R13: 510Ω, PCM_JLCPCB:R_0402, F.Cu at (173.6, 117.5)
- added R14: 10kΩ, PCM_JLCPCB:R_0402, F.Cu at (162.8, 116.3)
- added R18: 10kΩ, PCM_JLCPCB:R_0402, F.Cu at (147.3, 119.3)
- added R19: 10kΩ, PCM_JLCPCB:R_0402, F.Cu at (147.3, 120.3)
- added R20: 10kΩ, PCM_JLCPCB:R_0402, F.Cu at (147.3, 117.2)
- added R50: 33kΩ, PCM_JLCPCB:R_0402, F.Cu at (29.4, 23.9)
- added R69: 330Ω, PCM_JLCPCB:R_0402, F.Cu at (54.9, 45.6)
- added R70: 47Ω, PCM_JLCPCB:R_0402, F.Cu at (54.9, 47.4)
- added R71: 10kΩ, PCM_JLCPCB:R_0402, F.Cu at (162.7, 90.9)
- added R72: 10kΩ, PCM_JLCPCB:R_0402, F.Cu at (162.7, 92.8)
- added R73: 10kΩ, PCM_JLCPCB:R_0402, F.Cu at (15.4, 53.1)
- added R74: 1kΩ, PCM_JLCPCB:R_0402, F.Cu at (15.4, 54.9)
- added R75: 100Ω, PCM_JLCPCB:R_0603, F.Cu at (20.9, 39.8)
- added R77: 330Ω, PCM_JLCPCB:R_0402, F.Cu at (15.4, 56.8)
- added R78: 100Ω, PCM_JLCPCB:R_0603, F.Cu at (54.7, 34.6)
- added R79: 10kΩ, PCM_JLCPCB:R_0402, F.Cu at (54.9, 49.3)
- added R80: 47Ω, PCM_JLCPCB:R_0402, F.Cu at (18.2, 51.2)
- added R81: 100Ω, PCM_JLCPCB:R_0603, F.Cu at (20.9, 42.1)
- added R82: 10kΩ, PCM_JLCPCB:R_0402, F.Cu at (18.2, 53.1)
- added R83: 1kΩ, PCM_JLCPCB:R_0402, F.Cu at (18.2, 54.9)
- added R85: 330Ω, PCM_JLCPCB:R_0402, F.Cu at (18.2, 56.8)
- added R86: 47Ω, PCM_JLCPCB:R_0402, F.Cu at (21.1, 51.2)
- added R87: 1kΩ, PCM_JLCPCB:R_0402, F.Cu at (21.1, 53.1)
- added R89: 330Ω, PCM_JLCPCB:R_0402, F.Cu at (21.1, 54.9)
- added R90: 47Ω, PCM_JLCPCB:R_0402, F.Cu at (21.1, 56.8)
- added TP1: TestPoint, TestPoint:TestPoint_Pad_D1.0mm, F.Cu at (9.46, 24.7)
- added U3: M24C64, PCM_JLCPCB:SOIC-8_L5.0-W4.0-P1.27-LS6.0-BL, F.Cu at (61.6, 3.69)
- added X1: X322525MOB4SI, PCM_JLCPCB:OSC-SMD_4P-L3.2-W2.5-BL, F.Cu at (47.5, 68.5)
- C1, C2: value 100nF -> 10uF
- C16, C19: value 10uF -> 100nF
- C17, C18: value 10uF -> 12pF
- C4, C5: value 12pF -> 100nF
- D1: value M7 -> Red; footprint PCM_JLCPCB:D_SMA -> PCM_JLCPCB:D_0603
- D4: value SS510C -> Red; footprint SS510C:SMC_L7.1-W6.2-LS8.1-RD -> PCM_JLCPCB:D_0603
- D6: footprint SS510C:SMC_L7.1-W6.2-LS8.1-RD -> PCM_JLCPCB:D_SMC
- J7: value Program -> Conn_01x03_Pin
- J9: value LED connector -> Program; footprint Connector_JST:JST_XH_S4B-XH-A_1x04_P2.50mm_Horizontal -> Connector_PinHeader_2.54mm:PinHeader_1x03_P2.54mm_Vertical
- Q10, Q11, Q14, Q15, Q3, Q7, Q8: value 2N7002K -> MMBT2222A 1P
- Q12, Q4, Q9: value 2N7002K -> MMBT5401 200-300
- Q13, Q6: value 2N7002K -> AO3400A
- R15, R16: value 510Ω -> 10kΩ
- R21, R22: value 33kΩ -> 10kΩ
- R23: value 1kΩ -> 10kΩ
- R24: value 18.7k -> 10kΩ
- R25: value 16.5k -> 10kΩ
- R26: value 9.53k -> 10kΩ
- R27: value 5.11k -> 1kΩ
- R28: value 33kΩ -> 100Ω; footprint PCM_JLCPCB:R_0402 -> PCM_JLCPCB:R_0603
- R30, R38, R42, R52: value 10kΩ -> 330Ω
- R31: value 330Ω -> 100Ω; footprint PCM_JLCPCB:R_0402 -> PCM_JLCPCB:R_0603
- R32, R51, R53, R59: value 200Ω -> 10kΩ; footprint PCM_JLCPCB:R_0603 -> PCM_JLCPCB:R_0402
- R33, R39, R43, R60, R66: value 10kΩ -> 47Ω
- R34, R55, R61: value 200Ω -> 100Ω
- R36, R40, R54: value 10kΩ -> 1kΩ
- R44, R45, R47: value 10kΩ -> 33kΩ
- R46: value 10kΩ -> 3.9kΩ
- R48: value 10kΩ -> 1.2kΩ
- R49: value 200Ω -> 33kΩ; footprint PCM_JLCPCB:R_0603 -> PCM_JLCPCB:R_0402
- R57, R65: value 200Ω -> 330Ω; footprint PCM_JLCPCB:R_0603 -> PCM_JLCPCB:R_0402
- R58: value 10kΩ -> 100Ω; footprint PCM_JLCPCB:R_0402 -> PCM_JLCPCB:R_0603
- R63, R67: value 200Ω -> 1kΩ; footprint PCM_JLCPCB:R_0603 -> PCM_JLCPCB:R_0402
- U1: value SN74CB3Q3384APW -> AMS1117; footprint Package_SO:TSSOP-24_4.4x7.8mm_P0.65mm -> PCM_JLCPCB:SOT-223-3_L6.5-W3.4-P2.30-LS7.0-BR
- U2: value M24C64 -> SN74CB3Q3384APW; footprint PCM_JLCPCB:SOIC-8_L5.0-W4.0-P1.27-LS6.0-BL -> Package_SO:TSSOP-24_4.4x7.8mm_P0.65mm
- U4: value AMS1117 -> PCA9685PW,118; footprint PCM_JLCPCB:SOT-223-3_L6.5-W3.4-P2.30-LS7.0-BR -> easyeda2kicad:TSSOP-28_L9.7-W4.4-P0.65-LS6.4-TL
- U6: value AMS1117 -> LM2596HVS-ADJRG; footprint PCM_JLCPCB:SOT-223-3_L6.5-W3.4-P2.30-LS7.0-BR -> Package_TO_SOT_SMD:TO-263-5_TabPin3
- U7: value LM2596HVS-ADJRG -> CH32V003FxPx; footprint Package_TO_SOT_SMD:TO-263-5_TabPin3 -> PCM_JLCPCB:TSSOP-20_4.4x6.5mm_P0.65mm
- moved J7 264.7 mm to (5.64, 25.5)
- moved R47 245.6 mm to (29.4, 18.3)
- moved Q6 242.1 mm to (1.95, 38.9)
- moved R49 242.0 mm to (29.4, 22.0)
- moved S1 240.1 mm to (41.4, 68.6)
- moved R59 239.2 mm to (15.4, 51.2)
- moved J9 237.0 mm to (35.6, 60.7)
- moved R58 235.8 mm to (20.9, 37.6)
- moved Q3 230.8 mm to (35.7, 11.2)
- moved Q4 227.8 mm to (40.6, 1.90)
- moved Q8 227.1 mm to (40.6, 11.2)
- moved R31 226.2 mm to (54.7, 2.88)
- moved R30 225.5 mm to (49.2, 18.0)
- moved R44 223.8 mm to (29.4, 12.8)
- moved R45 223.8 mm to (29.4, 14.6)
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Connections:
- C1 pad 1: +3V3 -> +5V
- C16 pad 1: +5V -> +3V3
- C17 pad 1: +5V -> /CH32V003/OSCI
- C18 pad 1: +3V3 -> /CH32V003/OSCO
- C19 pad 1: +3V3 -> U_reg
- C20 pad 1: /Buck Regulator/sw-vin -> U_reg
- C20 pad 2: Net-(C20-Pad2) -> GND
- C4 pad 1: /CH32V003/OSCO -> +3V3
- C5 pad 1: /CH32V003/OSCI -> +5V
- C6 pad 1: +3V3 -> U_reg
- D1 pad 1: VIN_CHAINBUS -> Net-(D1-Pad1)
- D1 pad 2: /Buck Regulator/VIN_BRD -> +3V3
- D3 pad 1: Net-(D3-Pad1) -> GND
- D3 pad 2: +3V3 -> Net-(D3-Pad2)
- D4 pad 1: /Buck Regulator/sw -> GND
- D4 pad 2: GND -> Net-(D4-Pad2)
- D6 pad 1: Net-(D5-A) -> /Buck Regulator/sw
- D6 pad 2: Net-(D6-A) -> GND
- J1 pad 18: /Bus_switch/Chainbus_In.SDA -> /Interboard_connector/Chainbus.SDA
- J1 pad 20: /Bus_switch/Chainbus_In.SCL -> /Interboard_connector/Chainbus.SCL
- J1 pad 22: /Bus_switch/Chainbus_In.CS -> /Interboard_connector/Chainbus.CS
- J1 pad 24: /Bus_switch/Chainbus_In.SCK -> /Interboard_connector/Chainbus.SCK
- J1 pad 26: /Bus_switch/Chainbus_In.MOSI -> /Interboard_connector/Chainbus.MOSI
- J1 pad 28: /Bus_switch/Chainbus_In.MISO -> /Interboard_connector/Chainbus.MISO
- J1 pad 30: /Bus_switch/Chainbus_In.TX -> /Interboard_connector/Chainbus.TX
- J1 pad 32: /Bus_switch/Chainbus_In.RX -> /Interboard_connector/Chainbus.RX
- J10 pad 2: /LEDController1/Rin -> /LEDController/Rin
- J10 pad 3: /LEDController1/Gin -> /LEDController/Gin
- J10 pad 4: /LEDController1/Bin -> /LEDController/Bin
- J2 pad 18: /Bus_switch/Chainbus_In.SDA -> /Interboard_connector/Chainbus.SDA
- J2 pad 20: /Bus_switch/Chainbus_In.SCL -> /Interboard_connector/Chainbus.SCL
- J2 pad 22: /Bus_switch/Chainbus_In.CS -> /Interboard_connector/Chainbus.CS
- J2 pad 24: /Bus_switch/Chainbus_In.SCK -> /Interboard_connector/Chainbus.SCK
- J2 pad 26: /Bus_switch/Chainbus_In.MOSI -> /Interboard_connector/Chainbus.MOSI
- J2 pad 28: /Bus_switch/Chainbus_In.MISO -> /Interboard_connector/Chainbus.MISO
- J2 pad 30: /Bus_switch/Chainbus_In.TX -> /Interboard_connector/Chainbus.TX
- J2 pad 32: /Bus_switch/Chainbus_In.RX -> /Interboard_connector/Chainbus.RX
- J3 pad 1: /Chainbus.SDA -> /Bus_switch/Chainbus.SDA
- J3 pad 2: /Chainbus.SCL -> /Bus_switch/Chainbus.SCL
- J7 pad 1: GND -> /Buck Regulator/sw-vin
- J7 pad 2: /CH32V003/SWIO -> /Buck Regulator/VIN_BRD
- J7 pad 3: +3V3 -> /12V
- J9 pad 1: U_reg -> GND
- J9 pad 2: /LEDController/Rin -> /CH32V003/SWIO
- J9 pad 3: /LEDController/Gin -> +3V3
- L1 pad 2: U_reg -> /12V
- Q10 pad 1: Net-(Q10-G) -> Net-(Q10-B)
- Q10 pad 3: /LEDController2/Rin -> Net-(Q10-C)
- Q11 pad 1: Net-(Q11-G) -> Net-(Q10-C)
- Q11 pad 2: GND -> Net-(Q11-E)
- Q11 pad 3: /LEDController2/Gin -> /12V
- Q12 pad 1: Net-(Q12-G) -> Net-(Q10-C)
- Q12 pad 3: /LEDController2/Bin -> Net-(Q11-E)
- Q13 pad 3: /LEDController3/Rin -> /LEDController1/Gin
- Q14 pad 1: Net-(Q14-G) -> Net-(Q14-B)
- Q14 pad 3: /LEDController3/Gin -> Net-(Q14-C)
- Q15 pad 1: Net-(Q15-G) -> Net-(Q14-C)
- Q15 pad 2: GND -> Net-(Q15-E)
- Q15 pad 3: /LEDController3/Bin -> /12V
- Q3 pad 1: Net-(Q3-G) -> Net-(Q2-C)
- Q3 pad 2: GND -> Net-(Q3-E)
- Q3 pad 3: /LEDController/Rin -> /12V
- Q4 pad 1: Net-(Q4-G) -> Net-(Q2-C)
- Q4 pad 3: /LEDController/Gin -> Net-(Q3-E)
- Q6 pad 3: /LEDController1/Rin -> /LEDController2/Rin
- Q7 pad 1: Net-(Q7-G) -> Net-(Q7-B)
- Q7 pad 3: /LEDController1/Gin -> Net-(Q7-C)
- Q8 pad 1: Net-(Q8-G) -> Net-(Q7-C)
- Q8 pad 2: GND -> Net-(Q8-E)
- Q8 pad 3: /LEDController/Bin -> /12V
- Q9 pad 1: Net-(Q9-G) -> Net-(Q7-C)
- Q9 pad 3: /LEDController1/Bin -> Net-(Q8-E)
- R15 pad 1: /LED_IC/S15 -> /LED_IC/A5
- R15 pad 2: Net-(D8-Pad2) -> GND
- R16 pad 1: /LED_IC/S16 -> +5V
- R16 pad 2: Net-(D9-Pad2) -> /LED_IC/A4
- R17 pad 1: +3V3 -> /LED_IC/A4
- R17 pad 2: /CH32V003/PD7 -> GND
- R21 pad 1: /Buck Regulator/sw-vin -> /LED_IC/A2
- R21 pad 2: Net-(C20-Pad2) -> GND
- R22 pad 1: Net-(C20-Pad2) -> +5V
- R22 pad 2: GND -> /LED_IC/A1
- R23 pad 1: GND -> /LED_IC/A1
- R23 pad 2: Net-(U7-FB) -> GND
- R24 pad 1: Net-(U7-FB) -> +5V
- R24 pad 2: U_reg -> /LED_IC/A0
- R25 pad 1: Net-(R25-Pad1) -> /LED_IC/A0
- R25 pad 2: U_reg -> GND
- R26 pad 1: Net-(R26-Pad1) -> GND
- R26 pad 2: U_reg -> /LEDController1/S1
- R27 pad 1: Net-(R27-Pad1) -> /R2
- R27 pad 2: U_reg -> Net-(Q2-B)
- R28 pad 1: U_reg -> /LEDController1/S1
- R30 pad 1: /LEDController/R -> /12V
- R30 pad 2: GND -> Net-(Q2-C)
- R31 pad 1: /CH32V003/CH32V003.RX -> /LEDController1/S2
- R31 pad 2: Net-(D7-Pad2) -> Net-(Q13-G)
- R32 pad 1: /LEDController/R -> GND
- R32 pad 2: Net-(Q3-G) -> /LEDController1/S2
- R33 pad 1: /LEDController/G -> Net-(Q3-E)
- R33 pad 2: GND -> /LEDController1/S1
- R34 pad 1: /LEDController/G -> /LEDController/S2
- R34 pad 2: Net-(Q4-G) -> Net-(Q17-G)
- R35 pad 1: +5V -> GND
- R35 pad 2: /LED_IC/A5 -> /LEDController/S2
- R36 pad 1: /LED_IC/A5 -> /G2
- R36 pad 2: GND -> Net-(Q7-B)
- R38 pad 1: /LED_IC/A4 -> /12V
- R38 pad 2: GND -> Net-(Q7-C)
- R39 pad 1: +5V -> Net-(Q8-E)
- R39 pad 2: /LED_IC/A3 -> /LEDController1/S2
- R4 pad 1: /Bus_switch/SEL1 -> +3V3
- R4 pad 2: +3V3 -> /Bus_switch/Chainbus.SCL
- R40 pad 1: /LED_IC/A3 -> /B2
- R40 pad 2: GND -> Net-(Q10-B)
- R42 pad 1: /LED_IC/A2 -> /12V
- R42 pad 2: GND -> Net-(Q10-C)
- R43 pad 1: +5V -> Net-(Q11-E)
- R43 pad 2: /LED_IC/A1 -> /LEDController1/S3
- R44 pad 1: /LED_IC/A1 -> /Buck Regulator/sw-vin
- R44 pad 2: GND -> Net-(C10-Pad2)
- R45 pad 1: +5V -> Net-(C10-Pad2)
- R45 pad 2: /LED_IC/A0 -> GND
- R46 pad 1: /LED_IC/A0 -> GND
- R46 pad 2: GND -> Net-(U6-FB)
- R47 pad 1: /R1 -> Net-(U6-FB)
- R47 pad 2: GND -> Net-(R47-Pad2)
- R48 pad 1: /LEDController1/R -> Net-(R47-Pad2)
- R48 pad 2: GND -> /12V
- R49 pad 1: /R1 -> /12V
- R49 pad 2: Net-(Q8-G) -> Net-(C13-Pad2)
- R51 pad 1: /LEDController1/R -> +3V3
- R51 pad 2: Net-(Q6-G) -> /CH32V003/PD7
- R52 pad 1: /LEDController1/G -> /CH32V003/CH32V003.RX
- R52 pad 2: GND -> Net-(D9-Pad2)
- R53 pad 1: /LEDController1/G -> GND
- R53 pad 2: Net-(Q7-G) -> /LEDController/S1
- R54 pad 1: /LEDController1/B -> /R1
- R54 pad 2: GND -> Net-(Q14-B)
- R55 pad 1: /LEDController1/B -> /LEDController/S1
- R55 pad 2: Net-(Q9-G) -> Net-(Q5-G)
- R57 pad 1: /LEDController2/R -> /12V
- R57 pad 2: Net-(Q10-G) -> Net-(Q14-C)
- R58 pad 1: /LEDController2/G -> /LEDController2/S2
- R58 pad 2: GND -> Net-(Q18-G)
- R59 pad 1: /LEDController2/G -> GND
- R59 pad 2: Net-(Q11-G) -> /LEDController2/S2
- R60 pad 1: /LEDController2/B -> Net-(Q15-E)
- R60 pad 2: GND -> /LEDController/S1
- R61 pad 1: /LEDController2/B -> /LEDController1/S3
- R61 pad 2: Net-(Q12-G) -> Net-(Q27-G)
- R62 pad 1: /LEDController3/R -> GND
- R62 pad 2: GND -> /LEDController1/S3
- R63 pad 1: /LEDController3/R -> /G1
- R63 pad 2: Net-(Q13-G) -> Net-(Q19-B)
- R65 pad 1: /LEDController3/G -> /12V
- R65 pad 2: Net-(Q14-G) -> Net-(Q19-C)
- R66 pad 1: /LEDController3/B -> Net-(Q20-E)
- R66 pad 2: GND -> /LEDController/S2
- R67 pad 1: /LEDController3/B -> /B1
- R67 pad 2: Net-(Q15-G) -> Net-(Q22-B)
- R8 pad 2: /Bus_switch/Chainbus.RX -> /Bus_switch/Chainbus.SDA
- U1 pad 1: /Bus_switch/SEL1 -> GND
- U1 pad 2: /Bus_switch/Chainbus.RX -> +3V3
- U1 pad 3: /Bus_switch/Chainbus_In.RX -> +5V
- U1 pad 4: /Bus_switch/Chainbus_In.TX -> +3V3
- U2 pad 1: GND -> /Bus_switch/SEL1
- U2 pad 2: GND -> /Bus_switch/Chainbus.RX
- U2 pad 3: GND -> /Bus_switch/Chainbus_In.RX
- U2 pad 4: GND -> /Bus_switch/Chainbus_In.TX
- U2 pad 5: /Chainbus.SDA -> /Bus_switch/Chainbus.TX
- U2 pad 6: /Chainbus.SCL -> /Bus_switch/Chainbus.MISO
- U2 pad 7: unconnected-(U2-#WC-Pad7) -> /Bus_switch/Chainbus_In.MISO
- U2 pad 8: +3V3 -> /Bus_switch/Chainbus_In.MOSI
- U4 pad 1: GND -> /LED_IC/A0
- U4 pad 2: +3V3 -> /LED_IC/A1
- U4 pad 3: +5V -> /LED_IC/A2
- U4 pad 4: +3V3 -> /LED_IC/A3
- U6 pad 1: GND -> /Buck Regulator/sw-vin
- U6 pad 2: +3V3 -> /Buck Regulator/sw
- U6 pad 3: +5V -> GND
- U6 pad 4: +3V3 -> Net-(U6-FB)
- U7 pad 1: /Buck Regulator/sw-vin -> /B1
- U7 pad 2: /Buck Regulator/sw -> /CH32V003/CH32V003.TX
- U7 pad 3: GND -> /CH32V003/CH32V003.RX
- U7 pad 4: Net-(U7-FB) -> /CH32V003/PD7
- U7 pad 5: GND -> /CH32V003/OSCI
Routing:
- net /Bus_switch/SEL1: track 108.6 -> 0.00 mm, vias 4 -> 0
- net +5V: track 62.5 -> 0.69 mm, vias 7 -> 3
- net U_reg: track 61.4 -> 0.00 mm
- net +3V3: track 59.0 -> 0.00 mm, vias 4 -> 0
- net GND: track 57.7 -> 0.00 mm, vias 71 -> 18
- net (no net): track 55.6 -> 0.00 mm, vias 35 -> 0
- net /Chainbus.SDA: track 38.9 -> 0.00 mm, vias 2 -> 0
- net /Chainbus.SCL: track 35.6 -> 0.00 mm
- net VIN_CHAINBUS: track 33.7 -> 0.76 mm
- net /Buck Regulator/VIN_BRD: track 32.6 -> 0.00 mm
- net /Bus_switch/Chainbus_In.SDA: track 20.4 -> 0.00 mm, vias 2 -> 0
- net /Bus_switch/Chainbus_In.SCL: track 18.6 -> 0.00 mm, vias 2 -> 0
- net /Bus_switch/Chainbus_In.CS: track 14.2 -> 0.00 mm, vias 1 -> 0
- net Vin: track 12.5 -> 0.00 mm
- net Net-(D5-A): track 11.6 -> 0.00 mm
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- removed copper zone on B.Cu, net (none)
- removed copper zone on F.Cu, net (none)
- removed copper zone on F.Cu, net /Buck Regulator/sw
- removed copper zone on F.Cu, net /Buck Regulator/sw-vin
- removed copper zone on F.Cu, net Net-(C20-Pad2)
- removed copper zone on F.Cu, net Net-(Q1-G)
- removed copper zone on F.Cu, net U_reg
Other:
- board text removed: "3V3"
- board text removed: "GND"
- board text removed: "J1"
- board text removed: "J2"
- board text removed: "SCL"
- board text removed: "SDA"
- board text removed: "SEL LED"
