File: Hardware/CH32V003.kicad_sch (KiCad schematic)
At the start: 11 parts, among them J8 WCH Link, J9 Program, U7 CH32V003FxPx, X1 X322525MOB4SI

Commit message: updated readme
Connections:
- net GND: now also J9.2 (Pin_2); no longer J9.1 (Pin_1)
- net SWIO: now also J9.1 (Pin_1); no longer J9.2 (Pin_2)
Changed lines of the file:
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@@
 	)
 	(label "SWIO"
-		(at 58.42 134.62 180)
+		(at 53.34 132.08 180)
 		(effects
 			(font
@@
 	(symbol
 		(lib_id "power:GND")
-		(at 53.34 132.08 270)
+		(at 58.42 134.62 270)
 		(unit 1)
 		(body_style 1)
@@
 		(dnp no)
 		(property "Reference" "#PWR0103"
-			(at 46.99 132.08 0)
+			(at 52.07 134.62 0)
 			(hide yes)
 			(show_name no)
@@
 		)
 		(property "Value" "GND"
-			(at 46.482 132.08 90)
+			(at 51.562 134.62 90)
 			(show_name no)
 			(do_not_autoplace no)
@@
 		)
 		(property "Footprint" ""
-			(at 53.34 132.08 0)
+			(at 58.42 134.62 0)
 			(hide yes)
 			(show_name no)
@@
 		)
 		(property "Datasheet" ""
-			(at 53.34 132.08 0)
+			(at 58.42 134.62 0)
 			(hide yes)
 			(show_name no)
@@
 		)
 		(property "Description" "Power symbol creates a global label with name \"GND\" , ground"
-			(at 53.34 132.08 0)
-			(hide yes)
-			(show_name no)
+			(at 58.42 134.62 0)
+			(hide yes)
+			(show_name no)
