File: Hardware/LEDController.kicad_sch (KiCad schematic)
At the start: 29 parts, among them J6 LED connector, Q1 AO3400A, Q10 MMBT2222A 1P, Q11 MMBT2222A 1P, Q12 MMBT5401 200-300, Q13 AO3400A, Q2 MMBT2222A 1P, Q27 AO3400A, Q3 MMBT2222A 1P, Q4 MMBT5401 200-300, Q7 MMBT2222A 1P, Q8 MMBT2222A 1P, Q9 MMBT5401 200-300

Commit message: updated readme
Changed lines of the file:
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@@
 	(text "IC control\n\n"
 		(exclude_from_sim no)
-		(at 27.686 18.034 0)
+		(at 26.924 20.066 0)
 		(effects
 			(font
